File: AirCube/aircube.kicad_pcb (KiCad board)
At the start: 4 copper layers, 0 parts

Commit message: wip
Parts:
- added C1: 4u7, Capacitor_SMD:C_0603_1608Metric, F.Cu at (250.8, 64.8)
- added C2: 4u7, Capacitor_SMD:C_0603_1608Metric, F.Cu at (250.8, 67.3)
- added C4: 100n, Capacitor_SMD:C_0603_1608Metric, F.Cu at (250.8, 69.8)
- added C5: 1u, Capacitor_SMD:C_0603_1608Metric, F.Cu at (250.8, 72.3)
- added C6: 100n, Capacitor_SMD:C_0603_1608Metric, F.Cu at (250.8, 74.8)
- added C7: 100n, Capacitor_SMD:C_0603_1608Metric, F.Cu at (200.5, 76.8)
- added C8: 100n, Capacitor_SMD:C_0603_1608Metric, F.Cu at (200.5, 79.3)
- added F1: Polyfuse, Fuse:Fuse_1812_4532Metric, F.Cu at (236.2, 99.6)
- added J2: Conn_01x04, Connector_PinHeader_2.54mm:PinHeader_1x04_P2.54mm_Vertical, F.Cu at (221.2, 98.7)
- added R1: 4k7, Resistor_SMD:R_0603_1608Metric, F.Cu at (250.8, 77.3)
- added R2: 4k7, Resistor_SMD:R_0603_1608Metric, F.Cu at (250.8, 79.8)
- added R3: 12k, Resistor_SMD:R_0603_1608Metric, F.Cu at (250.8, 82.3)
- added R4: 12k, Resistor_SMD:R_0603_1608Metric, F.Cu at (250.8, 84.8)
- added R5: 4k7, Resistor_SMD:R_0603_1608Metric, F.Cu at (200.5, 81.8)
- added R6: 4k7, Resistor_SMD:R_0603_1608Metric, F.Cu at (200.5, 84.3)
- added R7: 12k, Resistor_SMD:R_0603_1608Metric, F.Cu at (200.5, 86.8)
- added R8: 12k, Resistor_SMD:R_0603_1608Metric, F.Cu at (200.5, 89.3)
- added U1: ESP32-C6-MINI-1, RF_Module:ESP32-C6-MINI-1, F.Cu at (226.6, 90.0)
- added U2: AMS1117-3.3, Package_TO_SOT_SMD:SOT-223-3_TabPin2, F.Cu at (228.5, 100.6)
- added U3: USBLC6-2P6, Package_TO_SOT_SMD:SOT-666, F.Cu at (235.4, 104.5)
- added U4: BME680, Package_LGA:Bosch_LGA-8_3x3mm_P0.8mm_ClockwisePinNumbering, F.Cu at (191.8, 84.1)
- added USB1: UC09-0B16F00P11, lcsc_footprints:C36936538_USB-C_UC09-0B16F00P11, F.Cu at (208.9, 98.0)
Other:
- board outline added: 50 x 50 mm

Commit message: wip
Parts:
- removed J2: Conn_01x04, Connector_PinHeader_2.54mm:PinHeader_1x04_P2.54mm_Vertical
- added C10: 100n, Capacitor_SMD:C_0603_1608Metric, F.Cu at (247.2, 64.5)
- added C9: 100n, Capacitor_SMD:C_0603_1608Metric, F.Cu at (247.2, 62.0)
- added D1: WS2812B, LED_SMD:LED_WS2812B_PLCC4_5.0x5.0mm_P3.2mm, F.Cu at (151.9, 108.0)
- added D2: WS2812B, LED_SMD:LED_WS2812B_PLCC4_5.0x5.0mm_P3.2mm, F.Cu at (151.9, 99.0)
- added D3: RED, LED_SMD:LED_0603_1608Metric, F.Cu at (214.4, 69.0)
- added R10: 330, Resistor_SMD:R_0603_1608Metric, F.Cu at (247.2, 67.0)
- added R9: 330, Resistor_SMD:R_0603_1608Metric, F.Cu at (214.3, 71.6)
- F1: value Polyfuse -> Polyfuse 1A
- R1, R2: value 4k7 -> 5k1
- U4: value BME680 -> BME688
- moved F1 98.5 mm to (138.0, 92.0), turned to -90 degrees
- moved U2 94.9 mm to (135.0, 84.0), turned to 90 degrees
- moved USB1 76.9 mm to (132.0, 99.0), turned to -90 degrees
- moved U1 75.2 mm to (152.0, 81.1)
- moved U4 53.6 mm to (151.9, 120.0)
- moved C1 41.3 mm to (223.2, 95.5), turned to 90 degrees
- moved C2 37.7 mm to (225.7, 95.5), turned to 90 degrees
- moved C4 34.2 mm to (228.2, 95.5), turned to 90 degrees
- moved C5 30.6 mm to (230.7, 95.5), turned to 90 degrees
- moved C6 27.1 mm to (233.2, 95.5), turned to 90 degrees
- moved U3 26.5 mm to (230.2, 78.5)
- moved R1 23.6 mm to (235.8, 95.5), turned to 90 degrees
- moved R2 20.0 mm to (238.3, 95.5), turned to 90 degrees
- moved C7 18.0 mm to (215.5, 86.7)
- moved C8 18.0 mm to (215.5, 89.2)
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Connections:
- U1 pad 27: unconnected-(U1-IO21-Pad27) -> /WS2812_DIN
Routing:
- added copper zone on In1.Cu, net GND
- added copper zone on In2.Cu, net GND

Commit message: wip
Parts:
- added C11: 100n, Capacitor_SMD:C_0603_1608Metric, F.Cu at (161.3, 96.5)
- added H1: MountingHole_Pad, MountingHole:MountingHole_2.2mm_M2_Pad, F.Cu at (129.4, 76.5)
- added H2: MountingHole_Pad, MountingHole:MountingHole_2.2mm_M2_Pad, F.Cu at (184.6, 76.5)
- added H3: MountingHole_Pad, MountingHole:MountingHole_2.2mm_M2_Pad, F.Cu at (184.6, 131.6)
- added H4: MountingHole_Pad, MountingHole:MountingHole_2.2mm_M2_Pad, F.Cu at (129.4, 131.6)
- added J1: Conn_01x04, Connector_PinHeader_2.54mm:PinHeader_1x04_P2.54mm_Vertical, F.Cu at (169.5, 77.5)
- added J2: Conn_01x04, Connector_JST:JST_PH_B4B-PH-K_1x04_P2.00mm_Vertical, F.Cu at (131.4, 97.2)
- added R11: 10k, Resistor_SMD:R_0603_1608Metric, F.Cu at (160.2, 88.3)
- added R12: 33, Resistor_SMD:R_0603_1608Metric, F.Cu at (155.8, 88.3)
- added R13: 33, Resistor_SMD:R_0603_1608Metric, F.Cu at (157.4, 88.3)
- added R14: 0R, Resistor_SMD:R_1206_3216Metric, F.Cu at (136.4, 103.2)
- added R15: 0R, Resistor_SMD:R_1206_3216Metric, F.Cu at (136.4, 97.2)
- added U5: SN74LV1T34DBV, Package_TO_SOT_SMD:SOT-23-5, F.Cu at (158.3, 96.4)
- C4: value 100n -> 10u
- R3, R4: value 12k -> 10k
- R9: value 330 -> 330R
- moved C10 104.9 mm to (152.6, 109.8), turned to -90 degrees
- moved C9 103.6 mm to (152.6, 104.1), turned to -90 degrees
- moved R2 101.6 mm to (137.1, 86.9), turned to 0 degrees
- moved R1 99.5 mm to (137.1, 83.2), turned to 0 degrees
- moved R10 93.7 mm to (159.5, 99.7), turned to -90 degrees
- moved U3 93.3 mm to (137.1, 85.1)
- moved D3 87.9 mm to (129.6, 92.4)
- moved C6 86.6 mm to (148.5, 78.0)
- moved R9 84.4 mm to (132.6, 92.4), turned to 180 degrees
- moved C4 83.3 mm to (146.8, 78.0)
- moved C1 82.9 mm to (140.7, 104.3), turned to 0 degrees
- moved C2 80.0 mm to (145.7, 95.0), turned to 180 degrees
- moved C7 53.3 mm to (198.4, 137.2), turned to 180 degrees
- moved C8 51.3 mm to (195.6, 136.5), turned to -90 degrees
- moved R6 49.8 mm to (166.5, 85.2)
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Connections:
- net Net-(U1-EN) renamed /~{RESET}
- net Net-(U1-IO9) renamed /BOOT
- net Net-(USB1-CC1) renamed /USB_CC1
- net Net-(USB1-CC2) renamed /USB_CC2
- D3 pad 1: Net-(D3-K) -> GND
- D3 pad 2: +5V -> Net-(D3-A)
- F1 pad 1: +5V -> VBUSF
- R10 pad 1: /WS2812_DIN -> Net-(U5-Y)
- R9 pad 1: Net-(D3-K) -> VBUSF
- R9 pad 2: GND -> Net-(D3-A)
- U1 pad 17: /USB_D- -> Net-(U1-IO12)
- U1 pad 18: /USB_D+ -> Net-(U1-IO13)
- U1 pad 22: unconnected-(U1-IO8-Pad22) -> /IO8
- U3 pad 1: Net-(USB1-Dn1) -> /USB_D-
- U3 pad 3: Net-(USB1-Dp1) -> /USB_D+
- U3 pad 4: /USB_D+ -> /USB_MCU_D+
- U3 pad 5: +5V -> VBUSF
- U3 pad 6: /USB_D- -> /USB_MCU_D-
- USB1 pad A6: Net-(USB1-Dp1) -> /USB_D+
- USB1 pad A7: Net-(USB1-Dn1) -> /USB_D-
- USB1 pad B6: Net-(USB1-Dp1) -> /USB_D+
- USB1 pad B7: Net-(USB1-Dn1) -> /USB_D-
Routing:
- net GND: track 0.00 -> 104.7 mm, vias 0 -> 27
- net +3V3: track 0.00 -> 85.1 mm, vias 0 -> 5
- net +5V: track 0.00 -> 55.1 mm, vias 0 -> 2
- net VBUSF: track 0.00 -> 25.2 mm, vias 0 -> 2
- net /WS2812_DIN: track 0.00 -> 19.5 mm, vias 0 -> 2
- net /UART_RX: track 0.00 -> 13.0 mm
- net VBUS: track 0.00 -> 10.4 mm
- net /UART_TX: track 0.00 -> 10.1 mm
- net Net-(D1-DOUT): track 0.00 -> 5.91 mm
- net /USB_D-: track 0.00 -> 4.85 mm
- net /I2C_SDA: track 0.00 -> 4.73 mm
- net /I2C_SCL: track 0.00 -> 4.72 mm
- net /USB_D+: track 0.00 -> 3.70 mm
- net /BAT_IN: track 0.00 -> 3.54 mm
- net /USB_CC1: track 0.00 -> 2.23 mm
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Other:
- board size 50 x 50 mm -> 60 x 60 mm

Commit message: wip
Parts:
- removed C1, C2: 4u7, Capacitor_SMD:C_0603_1608Metric
- removed R15: 0R, Resistor_SMD:R_1206_3216Metric
- added C12: 10u, Capacitor_SMD:C_0805_2012Metric, F.Cu at (145.2, 108.4)
- added C13: 100n, Capacitor_SMD:C_0603_1608Metric, F.Cu at (139.7, 107.8)
- added C14: 10u, Capacitor_SMD:C_0805_2012Metric, F.Cu at (143.4, 95.7)
- added C15: 10u, Capacitor_SMD:C_0805_2012Metric, F.Cu at (143.4, 97.7)
- added L2: ASPI-0628-3R9M-T1, lcsc_footprints:C5570229_IND-SMD_L6_0-W6_0, F.Cu at (141.0, 102.5)
- J2: value Conn_01x04 -> Conn_01x06; footprint Connector_JST:JST_PH_B4B-PH-K_1x04_P2.00mm_Vertical -> Connector_JST:JST_PH_B6B-PH-K_1x06_P2.00mm_Vertical
- R14: footprint Resistor_SMD:R_1206_3216Metric -> Resistor_SMD:R_0805_2012Metric_Pad1.20x1.40mm_HandSolder
- U2: value AMS1117-3.3 -> AP63203WU; footprint Package_TO_SOT_SMD:SOT-223-3_TabPin2 -> Package_TO_SOT_SMD:TSOT-23-6
- moved C5 69.5 mm to (148.5, 84.3)
- moved R3 69.5 mm to (148.5, 81.3)
- moved R8 51.6 mm to (182.0, 88.6), turned to 180 degrees
- moved C7 48.7 mm to (182.6, 91.1), turned to -90 degrees
- moved U4 47.1 mm to (179.9, 91.2), turned to 90 degrees
- moved C8 44.7 mm to (181.9, 93.9), turned to 0 degrees
- moved R7 44.1 mm to (177.3, 92.4), turned to 90 degrees
- moved R4 41.2 mm to (161.9, 88.3), turned to 90 degrees
- moved J2 12.9 mm to (130.5, 110.0), turned to 90 degrees
- moved U2 8.66 mm to (142.4, 108.4), turned to 90 degrees
- moved R14 5.02 mm to (135.0, 108.0), turned to -90 degrees
- moved R5 0.68 mm to (166.5, 82.8), turned to 90 degrees
- moved R6 0.61 mm to (166.5, 85.8), turned to -90 degrees
Connections:
- F1 pad 1: VBUSF -> VBUS
- F1 pad 2: VBUS -> Net-(F1-Pad2)
- J2 pad 1: /BAT_IN -> +5V
- J2 pad 3: GND -> VBUS
- J2 pad 4: +5V -> GND
- R14 pad 1: +5V -> VBUS
- R14 pad 2: VBUSF -> +5V
- R9 pad 1: VBUSF -> VBUS
- U2 pad 1: GND -> +3V3
- U2 pad 2: +3V3 -> +5V
- U3 pad 5: VBUSF -> VBUS
- USB1 pad A4B9: VBUS -> Net-(F1-Pad2)
- USB1 pad B4A9: VBUS -> Net-(F1-Pad2)
Routing:
- net /I2C_SDA: track 4.73 -> 67.7 mm
- net /I2C_SCL: track 4.72 -> 64.4 mm, vias 0 -> 2
- net VBUSF: track 25.2 -> 0.00 mm, vias 2 -> 0
- net VBUS: track 10.4 -> 35.3 mm, vias 0 -> 4
- net /USB_MCU_D+: track 0.00 -> 24.0 mm
- net /USB_MCU_D-: track 0.00 -> 23.2 mm
- net +5V: track 55.1 -> 42.2 mm, vias 2 -> 0
- net Net-(F1-Pad2): track 0.00 -> 10.4 mm
- net /BUCK_SW: track 0.00 -> 6.09 mm
- net GND: track 104.7 -> 100.3 mm, vias 27 -> 62
- net /BAT_IN: track 3.54 -> 0.00 mm
- net /~{RESET}: track 1.35 -> 4.03 mm
- net /BOOT: track 0.00 -> 2.23 mm
- net /WS2812_DIN: track 19.5 -> 21.7 mm, vias 2 -> 4
- net /BUCK_BST: track 0.00 -> 1.90 mm
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- added copper zone on F.Cu, net +3V3
- added copper zone on F.Cu, net +5V
- added copper zone on F.Cu, net GND
