File: AirCube/aircube.kicad_sch (KiCad schematic)
At the start: 18 parts, among them J1 Conn_01x04, J2 Connector, USB-TYPE-C-16P, U1 ESP32-C6-MINI-1, U2 AMS1117, U3 USBLC6-2SC6

Commit message: wip
Parts:
- removed C1, C2: 4.7uF, PCM_JLCPCB:C_0603, symbol PCM_JLCPCB-Capacitors:0603,4.7uF
- removed C3, C4: 100nF, PCM_JLCPCB:C_0603, symbol PCM_JLCPCB-Capacitors:0603,100nF
- removed C5: 1uF, PCM_JLCPCB:C_0603, symbol PCM_JLCPCB-Capacitors:0603,1uF
- removed F1: Fuse_Small, Fuse:Fuse_1812_4532Metric_Pad1.30x3.40mm_HandSolder, symbol Device:Fuse_Small
- removed J1: Conn_01x04, Connector_PinHeader_2.54mm:PinHeader_1x04_P2.54mm_Vertical, symbol Connector_Generic:Conn_01x04
- removed J2: Connector, USB-TYPE-C-16P, PCM_JLCPCB:TYPE-C-SMD_HX-TYPE-C-16PIN, symbol PCM_JLCPCB-Extended:Connector, USB-TYPE-C-16P
- removed R1, R2: 4.7kΩ, PCM_JLCPCB:R_0603, symbol PCM_JLCPCB-Resistors:0603,4.7kΩ
- removed R3, R4: 10kΩ, PCM_JLCPCB:R_0603, symbol PCM_JLCPCB-Resistors:0603,10kΩ
- removed R5: 0Ω, PCM_JLCPCB:R_0603, symbol PCM_JLCPCB-Resistors:0603,0Ω
- removed S1, S2: Tactile Button, 160gf, PCM_JLCPCB:SW_TS-1088-AR02016, symbol PCM_JLCPCB-Connectors_Buttons:Tactile Button, 160gf, 12V, 50mA, 4.0mm
- removed U2: AMS1117, PCM_JLCPCB:SOT-223-3_L6.5-W3.4-P2.30-LS7.0-BR, symbol PCM_JLCPCB-Power:LDO, 3.3V, 1A
- removed U3: USBLC6-2SC6, Package_TO_SOT_SMD:SOT-23-6, symbol Power_Protection:USBLC6-2SC6
- added C1, C2: 4u7, Capacitor_SMD:C_0603_1608Metric, symbol Device:C
- added C4, C6, C7, C8: 100n, Capacitor_SMD:C_0603_1608Metric, symbol Device:C
- added C5: 1u, Capacitor_SMD:C_0603_1608Metric, symbol Device:C
- added F1: Polyfuse, Fuse:Fuse_1812_4532Metric, symbol Device:Polyfuse
- added J2: Conn_01x04, Connector_PinHeader_2.54mm:PinHeader_1x04_P2.54mm_Vertical, symbol Connector_Generic:Conn_01x04
- added R1, R2, R5, R6: 4k7, Resistor_SMD:R_0603_1608Metric, symbol Device:R
- added R3, R4, R7, R8: 12k, Resistor_SMD:R_0603_1608Metric, symbol Device:R
- added SW1, SW2: SW_Push, symbol Switch:SW_Push
- added U2: AMS1117-3.3, Package_TO_SOT_SMD:SOT-223-3_TabPin2, symbol Regulator_Linear:AMS1117-3.3
- added U3: USBLC6-2P6, Package_TO_SOT_SMD:SOT-666, symbol Power_Protection:USBLC6-2P6
- added U4: BME680, Package_LGA:Bosch_LGA-8_3x3mm_P0.8mm_ClockwisePinNumbering, symbol Sensor:BME680
- added USB1: UC09-0B16F00P11, lcsc_footprints:C36936538_USB-C_UC09-0B16F00P11, symbol lcsc_imported:UC09-0B16F00P11
- U1: LCSC C5366877 -> (none)
Connections:
- net +3V3: now also C2.1, C4.1, C6.1, C7.1, C8.1, J2.1 (Pin_1), R3.1, R4.1, R5.2, R6.2, R7.1, R8.1, U2.2 (VO), U4.6 (VDDIO), U4.8 (VDD)
- net GND: now also C1.2, C2.2, C4.2, C5.2, C6.2, C7.2, C8.2, J2.4 (Pin_4), R1.2, R2.2, SW1.2, SW2.2, U2.1 (GND), U3.2 (GND), U4.1 (GND), U4.7 (GND), USB1.17 (EH), USB1.18 (EH), USB1.19 (EH), USB1.20 (EH), USB1.A1B12 (GND), USB1.B1A12 (GND)
- net USB_D+: now also U3.4 (I/O2)
- net USB_D-: now also U3.6 (I/O1)
- net VBUS: now also F1.2, USB1.A4B9 (VBUS), USB1.B4A9 (VBUS)
- net at U1.23 (IO9): now also R4.2, SW2.1
- net at U1.8 (EN): now also C5.1, R3.2, SW1.1
- net UART_TX: now reaches U1.31 (TXD0)
- net UART_TX: now also J2.2 (Pin_2)
- net UART_RX: now reaches U1.30 (RXD0)
- net UART_RX: now also J2.3 (Pin_3)
- net I2C_SCL: now reaches U1.25 (IO19)
- net I2C_SCL: now also R6.1, U4.4 (SCK)
- net I2C_SDA: now reaches U1.26 (IO20)
- net I2C_SDA: now also R5.1, U4.3 (SDI)
- new net: R7.2, U4.2 (CSB)
- new net: R8.2, U4.5 (SDO)
- new net: U3.1 (I/O1), USB1.A7 (Dn1), USB1.B7 (Dn2)
- new net: U3.3 (I/O2), USB1.A6 (Dp1), USB1.B6 (Dp2)
- new net: R1.1, USB1.A5 (CC1)
- new net: R2.1, USB1.B5 (CC2)
- new net +5V: C1.1, F1.1, U2.3 (VI), U3.5 (VBUS)
Other:
- note added: "BME688 I²C address select: SDO = GND -> 0x76 SDO = VDDIO -> 0x77"

Commit message: wip
Parts:
- removed J2: Conn_01x04, Connector_PinHeader_2.54mm:PinHeader_1x04_P2.54mm_Vertical, symbol Connector_Generic:Conn_01x04
- added C10, C9: 100n, Capacitor_SMD:C_0603_1608Metric, symbol Device:C
- added D1, D2: WS2812B, LED_SMD:LED_WS2812B_PLCC4_5.0x5.0mm_P3.2mm, symbol LED:WS2812B
- added D3: RED, LED_SMD:LED_0603_1608Metric, symbol Device:LED
- added J1: Conn_01x03, symbol Connector_Generic:Conn_01x03
- added R10, R9: 330, Resistor_SMD:R_0603_1608Metric, symbol Device:R
- F1: value Polyfuse -> Polyfuse 1A
- R1, R2: value 4k7 -> 5k1
- U4: value BME680 -> BME688
Connections:
- net +5V: now also C10.1, C9.1, D1.1 (VDD), D2.1 (VDD), D3.2 (A)
- net GND: now also C10.2, C9.2, D1.3 (VSS), D2.3 (VSS), J1.3 (Pin_3), R9.2
- net UART_RX: now also J1.2 (Pin_2)
- net UART_TX: now also J1.1 (Pin_1)
- net WS2812_DIN: now reaches U1.27 (IO21)
- net WS2812_DIN: now also R10.1
- new net: D3.1 (K), R9.1
- new net: D1.2 (DOUT), D2.4 (DIN)
- new net: D1.4 (DIN), R10.2
- no-connect marks 6 -> 7
Other:
- moved on the sheet: C1, C2, C4, C5, C6, F1, R1, R2, R3, R4, R5, R6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

Commit message: wip
Parts:
- removed J1: Conn_01x03, symbol Connector_Generic:Conn_01x03
- added C11: 100n, Capacitor_SMD:C_0603_1608Metric, symbol Device:C
- added H1, H2, H3, H4: MountingHole_Pad, MountingHole:MountingHole_2.2mm_M2_Pad, symbol Mechanical:MountingHole_Pad
- added J1: Conn_01x04, Connector_PinHeader_2.54mm:PinHeader_1x04_P2.54mm_Vertical, symbol Connector_Generic:Conn_01x04
- added NT1: NetTie_2, symbol Device:NetTie_2
- added R11: 10k, Resistor_SMD:R_0603_1608Metric, symbol Device:R
- added R12, R13: 33, Resistor_SMD:R_0603_1608Metric, symbol Device:R
- added U5: SN74LV1T34DBV, Package_TO_SOT_SMD:SOT-23-5, symbol Logic_LevelTranslator:SN74LV1T34DBV
- C4: value 100n -> 10u
- R3, R4: value 12k -> 10k
Connections:
- net +3V3: now also J1.1 (Pin_1), R11.1
- net +5V: now also C11.1, NT1.2, U5.5 (VCC); no longer D3.2 (A), F1.1, U3.5 (VBUS)
- net GND: now also C11.2, H1.1, H2.1, H3.1, H4.1, J1.4 (Pin_4), U5.3 (GND)
- net UART_RX: now also J1.3 (Pin_3)
- net UART_TX: now also J1.2 (Pin_2)
- net USB_D+: now also R13.1; no longer U1.18 (IO13)
- net USB_D-: now also R12.2; no longer U1.17 (IO12)
- net VBUS: now also D3.2 (A), F1.1, U3.5 (VBUS), NT1.1; no longer F1.2, USB1.A4B9 (VBUS), USB1.B4A9 (VBUS)
- net WS2812_DIN: now also U5.2 (A); no longer R10.1
- net ~{RESET}: now reaches C5.1, R3.2, SW1.1, U1.8 (EN)
- net BOOT: now reaches R4.2, SW2.1, U1.23 (IO9)
- net IO8: now reaches U1.22 (IO8)
- net IO8: now also R11.2
- new net: R10.1, U5.4 (Y)
- new net: R12.1, U1.17 (IO12)
- new net: F1.2, USB1.A4B9 (VBUS), USB1.B4A9 (VBUS)
- new net: R13.2, U1.18 (IO13)
- no-connect marks 7 -> 16
Other:
- note added: "3V3 Linear Regulator"
- note added: "BME688 I2C address select: SDO = GND -> 0x76 SDO = VDDIO -> 0x77"
- note added: "ESP32 MCU with WiFi, BLE, ZigBee and Thread"
- note added: "Fused USB-C Connector with Power LED"
- note added: "Keep this section far away from any heat emitting components. Ideally on its own island."
- note added: "Label pins on PCB!"
- note added: "RGB LED"
- note added: "Recommended 22R or 33R series resistors for USB."
- note added: "Recommended I2C pullup resistors at bus master."
- note added: "Temperature, Humidity and VOC Sensor"
- note added: "UART Header"
- note added: "WS2812 and similar RGB LEDs have a logic level of 0.7x for HIGH and 0.3x for LOW, requiring a level shifter for correct 3V3 communication."
- note removed: "BME688 I²C address select: SDO = GND -> 0x76 SDO = VDDIO -> 0x77"
- moved on the sheet: C10, C7, C8, C9, D1, D2, D3, F1, R1, R10, R2, R7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

Commit message: wip
Parts:
- removed NT1: NetTie_2, symbol Device:NetTie_2
- added J2: Conn_01x04, Connector_JST:JST_PH_B4B-PH-K_1x04_P2.00mm_Vertical, symbol Connector_Generic:Conn_01x04
- added R14, R15: 0R, Resistor_SMD:R_1206_3216Metric, symbol Device:R
- R9: value 330 -> 330R
Connections:
- net +5V: now also J2.4 (Pin_4), R14.1
- net GND: now also D3.1 (K), J2.2 (Pin_2), J2.3 (Pin_3); no longer R9.2
- net USB_D+: now also U3.3 (I/O2), USB1.A6 (Dp1), USB1.B6 (Dp2); no longer R13.1, U3.4 (I/O2)
- net USB_D-: now also U3.1 (I/O1), USB1.A7 (Dn1), USB1.B7 (Dn2); no longer R12.2, U3.6 (I/O1)
- net VBUS: now also F1.2, USB1.A4B9 (VBUS), USB1.B4A9 (VBUS); no longer D3.2 (A), F1.1, U3.5 (VBUS)
- net VBUSF: now reaches R9.1
- net VBUSF: now also F1.1, U3.5 (VBUS), R14.2, R15.2; no longer D3.1 (K)
- net USB_CC1: now reaches R1.1, USB1.A5 (CC1)
- net USB_CC2: now reaches R2.1, USB1.B5 (CC2)
- new net: D3.2 (A), R9.2
- new net BAT_IN: J2.1 (Pin_1), R15.1
- new net USB_MCU_D+: R13.1, U3.4 (I/O2)
- new net USB_MCU_D-: R12.2, U3.6 (I/O1)
Other:
- note added: "This connector is for a self-managed battery module. To enable, 0R resistor must be moved from +5V - VBUS bridge to the connector."
- moved on the sheet: D3, F1, R1, R2, R9, U3, USB1

Commit message: wip
Parts:
- removed C1, C2: 4u7, Capacitor_SMD:C_0603_1608Metric, symbol Device:C
- removed J2: Conn_01x04, Connector_JST:JST_PH_B4B-PH-K_1x04_P2.00mm_Vertical, symbol Connector_Generic:Conn_01x04
- removed R15: 0R, Resistor_SMD:R_1206_3216Metric, symbol Device:R
- removed U2: AMS1117-3.3, Package_TO_SOT_SMD:SOT-223-3_TabPin2, symbol Regulator_Linear:AMS1117-3.3
- added C12, C14, C15: 10u, Capacitor_SMD:C_0805_2012Metric, symbol Device:C
- added C13: 100n, Capacitor_SMD:C_0603_1608Metric, symbol Device:C
- added J2: Conn_01x06, Connector_JST:JST_PH_B6B-PH-K_1x06_P2.00mm_Vertical, symbol Connector_Generic:Conn_01x06
- added L2: ASPI-0628-3R9M-T1, lcsc_footprints:C5570229_IND-SMD_L6_0-W6_0, symbol lcsc_imported:ASPI-0628-3R9M-T1
- added U2: AP63203WU, Package_TO_SOT_SMD:TSOT-23-6, symbol Regulator_Switching:AP63203WU
- R14: footprint Resistor_SMD:R_1206_3216Metric -> Resistor_SMD:R_0805_2012Metric_Pad1.20x1.40mm_HandSolder
Connections:
- net +3V3: now also C14.1, C15.1, L2.2, U2.1 (FB)
- net +5V: now also R14.2, C12.1, J2.1 (Pin_1), U2.2 (EN), U2.3 (IN); no longer R14.1
- net GND: now also C12.2, C14.2, C15.2, J2.2 (Pin_2), J2.4 (Pin_4), U2.4 (GND)
- net I2C_SCL: now also J2.6 (Pin_6)
- net I2C_SDA: now also J2.5 (Pin_5)
- net VBUS: now also F1.1, R14.1, R9.1, U3.5 (VBUS), J2.3 (Pin_3); no longer F1.2, USB1.A4B9 (VBUS), USB1.B4A9 (VBUS)
- removed net VBUSF: F1.1, R14.2, R9.1, U3.5 (VBUS)
- new net: F1.2, USB1.A4B9 (VBUS), USB1.B4A9 (VBUS)
- new net BUCK_BST: C13.1, U2.6 (BST)
- new net BUCK_SW: C13.2, L2.1, U2.5 (SW)
Other:
- note added: "3V3 Switching Regulator"
- note added: "Protected USB-C Connector with Power LED"
- note added: "Smart Battery Connector"
- note added: "This is a connector for an optional battery module. The sensor module should not contain any battery logic in order to make it indepdent of any specific battery technology. The 0 Ohm resistor is used as a bypass if this connector is not used and should be desoldered / DNP if a battery module is used."
- note added: "This is a debug UART header. Its pins should be common pitch (2.54mm) and labeled on the PCB."
- note removed: "3V3 Linear Regulator"
- note removed: "Fused USB-C Connector with Power LED"
- note removed: "Label pins on PCB!"
- note removed: "This connector is for a self-managed battery module. To enable, 0R resistor must be moved from +5V - VBUS bridge to the connector."
- title: (none) -> AirCube
- moved on the sheet: D3, F1, J1, R1, R2, R9
